Commit message: Use full Picker meshes in simulation

File: .devcontainer/src/dfl_manipulation_toolbox/urdf/dfl_robot.urdf.xacro (robot description, xacro)
@@ -18,10 +18,20 @@
   <xacro:if value="${robot_id.startswith('picker')}">
     <link name="base_footprint">
-      <inertial><mass value="65"/><origin xyz="0 0 0.18"/><inertia ixx="4.0" ixy="0" ixz="0" iyy="4.0" iyz="0" izz="6.0"/></inertial>
-      <visual><origin xyz="0 0 0.18"/><geometry><box size="0.72 0.55 0.36"/></geometry><material name="picker_base"><color rgba="0.15 0.18 0.22 1"/></material></visual>
-      <collision><origin xyz="0 0 0.18"/><geometry><box size="0.72 0.55 0.36"/></geometry></collision>
+      <xacro:if value="${robot_id == 'picker1'}">
+        <inertial><mass value="65"/><origin xyz="0 0 0.295"/><inertia ixx="4.0" ixy="0" ixz="0" iyy="4.0" iyz="0" izz="6.0"/></inertial>
+        <visual><origin xyz="0 0 0.145" rpy="1.5708 0 0"/><geometry><mesh filename="package://dfl_manipulation_toolbox/meshes/picker1/base.stl"/></geometry><material name="picker_base"><color rgba="0.15 0.18 0.22 1"/></material></visual>
+        <visual><origin xyz="-0.25 0 0.4925"/><geometry><box size="0.50 0.70 0.405"/></geometry><material name="picker_pedestal"><color rgba="0.75 0.75 0.75 1"/></material></visual>
+        <collision><origin xyz="0 0 0.295"/><geometry><box size="0.85 0.65 0.30"/></geometry></collision>
+        <collision><origin xyz="-0.25 0 0.4925"/><geometry><box size="0.50 0.70 0.405"/></geometry></collision>
+      </xacro:if>
+      <xacro:if value="${robot_id == 'picker2'}">
+        <inertial><mass value="150.367639"/><origin xyz="0.0918 -0.0198 0.459"/><inertia ixx="60.652572" ixy="5.102762" ixz="-0.117004" iyy="46.813577" iyz="9.167281" izz="68.110164"/></inertial>
+        <visual><origin rpy="0 0 -1.5708"/><geometry><mesh filename="package://dfl_manipulation_toolbox/meshes/picker2/base.stl" scale="0.001 0.001 0.001"/></geometry><material name="picker_base"><color rgba="0.55 0.57 0.60 1"/></material></visual>
+        <collision><origin xyz="0.0918 -0.0198 0.43"/><geometry><box size="1.05 0.892 0.82"/></geometry></collision>
+      </xacro:if>
     </link>
     <joint name="world_to_base" type="fixed"><parent link="world"/><child link="base_footprint"/></joint>
-    <joint name="base_to_arm" type="fixed"><origin xyz="0 0 0.42"/><parent link="base_footprint"/><child link="base_link"/></joint>
+    <xacro:if value="${robot_id == 'picker1'}"><joint name="base_to_arm" type="fixed"><origin xyz="-0.165 0 0.695" rpy="0 0 -1.5708"/><parent link="base_footprint"/><child link="base_link"/></joint></xacro:if>
+    <xacro:if value="${robot_id == 'picker2'}"><joint name="base_to_arm" type="fixed"><origin xyz="-0.275 -0.020 0.876908"/><parent link="base_footprint"/><child link="base_link"/></joint></xacro:if>
   </xacro:if>
   <xacro:unless value="${robot_id.startswith('picker')}">
@@ -30,8 +40,8 @@
   <xacro:if value="${model == 'm1013'}"><xacro:m1013 namespace="${ns}" simple="true"/></xacro:if>
   <xacro:if value="${model == 'h2515'}"><xacro:h2515 namespace="${ns}" simple="true"/></xacro:if>
-  <xacro:macro name="box_tool" params="name mass size tcp_xyz body_xyz">
+  <xacro:macro name="box_tool" params="name mass size tcp_xyz body_xyz visual_mesh:=''">
     <link name="${name}_body">
       <inertial><mass value="${mass}"/><origin xyz="${body_xyz}"/><inertia ixx="0.002" ixy="0" ixz="0" iyy="0.002" iyz="0" izz="0.002"/></inertial>
-      <visual><origin xyz="${body_xyz}"/><geometry><box size="${size}"/></geometry><material name="tool_blue"><color rgba="0.08 0.32 0.70 1"/></material></visual>
+      <visual><geometry><xacro:if value="${visual_mesh != ''}"><mesh filename="${visual_mesh}"/></xacro:if><xacro:unless value="${visual_mesh != ''}"><box size="${size}"/></xacro:unless></geometry><material name="tool_blue"><color rgba="0.08 0.32 0.70 1"/></material></visual>
       <collision><origin xyz="${body_xyz}"/><geometry><box size="${size}"/></geometry></collision>
     </link>
@@ -40,12 +50,12 @@
   </xacro:macro>
   <xacro:if value="${tool_id == 'vgc10_1cup'}">
-    <link name="vgc10_1cup_body"><inertial><mass value="0.746664"/><origin xyz="0 0 0.0525"/><inertia ixx="0.001" ixy="0" ixz="0" iyy="0.001" iyz="0" izz="0.001"/></inertial><visual><origin xyz="0 0 0.0525"/><geometry><cylinder radius="0.05" length="0.105"/></geometry></visual><collision><origin xyz="0 0 0.0525"/><geometry><cylinder radius="0.05" length="0.105"/></geometry></collision></link>
+    <link name="vgc10_1cup_body"><inertial><mass value="0.746664"/><origin xyz="0 0 0.0525"/><inertia ixx="0.001" ixy="0" ixz="0" iyy="0.001" iyz="0" izz="0.001"/></inertial><visual><geometry><mesh filename="package://dfl_manipulation_toolbox/meshes/tools/vgc10_1cup.dae"/></geometry></visual><collision><origin xyz="0 0 0.0525"/><geometry><cylinder radius="0.05" length="0.105"/></geometry></collision></link>
     <joint name="vgc10_1cup_mount" type="fixed"><parent link="link_6"/><child link="vgc10_1cup_body"/></joint><link name="tool_tcp"/><joint name="vgc10_1cup_tcp" type="fixed"><origin xyz="0 0 0.17"/><parent link="vgc10_1cup_body"/><child link="tool_tcp"/></joint>
   </xacro:if>
-  <xacro:if value="${tool_id == 'vgc10_4cup'}"><xacro:box_tool name="vgc10_4cup" mass="0.746664" size="0.170 0.225 0.110" body_xyz="0 0 0.055" tcp_xyz="0 0 0.125"/></xacro:if>
-  <xacro:if value="${tool_id == 'vgp20'}"><xacro:box_tool name="vgp20" mass="2.77" size="0.145 0.105 0.100" body_xyz="0 0.04 0.05" tcp_xyz="0 0.04 0.10"/></xacro:if>
+  <xacro:if value="${tool_id == 'vgc10_4cup'}"><xacro:box_tool name="vgc10_4cup" mass="0.746664" size="0.170 0.225 0.110" body_xyz="0 0 0.055" tcp_xyz="0 0 0.125" visual_mesh="package://dfl_manipulation_toolbox/meshes/tools/vgc10_4cup.dae"/></xacro:if>
+  <xacro:if value="${tool_id == 'vgp20'}"><xacro:box_tool name="vgp20" mass="2.77" size="0.145 0.105 0.100" body_xyz="0 0.04 0.05" tcp_xyz="0 0.04 0.10" visual_mesh="package://dfl_manipulation_toolbox/meshes/tools/vgp20.dae"/></xacro:if>
   <xacro:if value="${tool_id == '2fg14'}"><xacro:box_tool name="2fg14" mass="1.5" size="0.115 0.070 0.1552" body_xyz="0 0 0.0776" tcp_xyz="0 0 0.136"/></xacro:if>
   <xacro:if value="${robot_id.startswith('picker')}">
-    <link name="camera_mount"/><joint name="camera_mount_joint" type="fixed"><origin xyz="0.05 0 0.10" rpy="0 0 0"/><parent link="link_6"/><child link="camera_mount"/></joint>
+    <link name="camera_mount"><visual><geometry><mesh filename="package://dfl_manipulation_toolbox/meshes/camera/hand_camera_mount.dae" scale="0.001 0.001 0.001"/></geometry></visual><collision><origin xyz="0 -0.0417 0.0105"/><geometry><box size="0.170 0.225 0.110"/></geometry></collision></link><joint name="camera_mount_joint" type="fixed"><origin xyz="0.05 0 0.10" rpy="0 0 0"/><parent link="link_6"/><child link="camera_mount"/></joint>
     <link name="camera_color_optical_frame"/><joint name="camera_optical_joint" type="fixed"><origin rpy="-1.5708 0 -1.5708"/><parent link="camera_mount"/><child link="camera_color_optical_frame"/></joint>
   </xacro:if>

Commit message: Add verified Genesis and Gazebo robot gallery

File: .devcontainer/src/dfl_manipulation_toolbox/urdf/dfl_robot.urdf.xacro (robot description, xacro)
@@ -40,5 +40,5 @@
   <xacro:if value="${model == 'm1013'}"><xacro:m1013 namespace="${ns}" simple="true"/></xacro:if>
   <xacro:if value="${model == 'h2515'}"><xacro:h2515 namespace="${ns}" simple="true"/></xacro:if>
-  <xacro:macro name="box_tool" params="name mass size tcp_xyz body_xyz visual_mesh:=''">
+  <xacro:macro name="box_tool" params="name mass size tcp_xyz body_xyz visual_mesh:='' mount_parent:='link_6' mount_xyz:='0 0 0'">
     <link name="${name}_body">
       <inertial><mass value="${mass}"/><origin xyz="${body_xyz}"/><inertia ixx="0.002" ixy="0" ixz="0" iyy="0.002" iyz="0" izz="0.002"/></inertial>
@@ -46,6 +46,18 @@
       <collision><origin xyz="${body_xyz}"/><geometry><box size="${size}"/></geometry></collision>
     </link>
-    <joint name="${name}_mount" type="fixed"><parent link="link_6"/><child link="${name}_body"/></joint>
+    <joint name="${name}_mount" type="fixed"><origin xyz="${mount_xyz}"/><parent link="${mount_parent}"/><child link="${name}_body"/></joint>
     <link name="tool_tcp"/><joint name="${name}_tcp" type="fixed"><origin xyz="${tcp_xyz}"/><parent link="${name}_body"/><child link="tool_tcp"/></joint>
+  </xacro:macro>
+  <!-- The source Picker assembly uses this D455-and-bracket CAD only with
+       tools that mount through the hand-camera plate.  It is not a generic
+       decoration and must stay in the tool's kinematic mounting chain. -->
+  <xacro:macro name="picker_hand_camera">
+    <link name="camera_mount">
+      <visual><geometry><mesh filename="package://dfl_manipulation_toolbox/meshes/camera/hand_camera_mount.dae" scale="0.001 0.001 0.001"/></geometry></visual>
+      <collision><origin xyz="0 -0.0417 0.0105"/><geometry><box size="0.104 0.155 0.043"/></geometry></collision>
+    </link>
+    <joint name="camera_mount_joint" type="fixed"><parent link="link_6"/><child link="camera_mount"/></joint>
+    <link name="camera_color_optical_frame"/>
+    <joint name="camera_optical_joint" type="fixed"><origin rpy="-1.5708 0 -1.5708"/><parent link="camera_mount"/><child link="camera_color_optical_frame"/></joint>
   </xacro:macro>
   <xacro:if value="${tool_id == 'vgc10_1cup'}">
@@ -53,10 +65,31 @@
     <joint name="vgc10_1cup_mount" type="fixed"><parent link="link_6"/><child link="vgc10_1cup_body"/></joint><link name="tool_tcp"/><joint name="vgc10_1cup_tcp" type="fixed"><origin xyz="0 0 0.17"/><parent link="vgc10_1cup_body"/><child link="tool_tcp"/></joint>
   </xacro:if>
-  <xacro:if value="${tool_id == 'vgc10_4cup'}"><xacro:box_tool name="vgc10_4cup" mass="0.746664" size="0.170 0.225 0.110" body_xyz="0 0 0.055" tcp_xyz="0 0 0.125" visual_mesh="package://dfl_manipulation_toolbox/meshes/tools/vgc10_4cup.dae"/></xacro:if>
+  <xacro:if value="${tool_id == 'vgc10_4cup'}">
+    <xacro:if value="${robot_id.startswith('picker')}">
+      <xacro:picker_hand_camera/>
+      <xacro:box_tool name="vgc10_4cup" mass="0.746664" size="0.170 0.225 0.110" body_xyz="0 0 0.055" tcp_xyz="0 0 0.125" visual_mesh="package://dfl_manipulation_toolbox/meshes/tools/vgc10_4cup.dae" mount_parent="camera_mount" mount_xyz="0 0 0.0125"/>
+    </xacro:if>
+    <xacro:unless value="${robot_id.startswith('picker')}"><xacro:box_tool name="vgc10_4cup" mass="0.746664" size="0.170 0.225 0.110" body_xyz="0 0 0.055" tcp_xyz="0 0 0.125" visual_mesh="package://dfl_manipulation_toolbox/meshes/tools/vgc10_4cup.dae"/></xacro:unless>
+  </xacro:if>
   <xacro:if value="${tool_id == 'vgp20'}"><xacro:box_tool name="vgp20" mass="2.77" size="0.145 0.105 0.100" body_xyz="0 0.04 0.05" tcp_xyz="0 0.04 0.10" visual_mesh="package://dfl_manipulation_toolbox/meshes/tools/vgp20.dae"/></xacro:if>
-  <xacro:if value="${tool_id == '2fg14'}"><xacro:box_tool name="2fg14" mass="1.5" size="0.115 0.070 0.1552" body_xyz="0 0 0.0776" tcp_xyz="0 0 0.136"/></xacro:if>
-  <xacro:if value="${robot_id.startswith('picker')}">
-    <link name="camera_mount"><visual><geometry><mesh filename="package://dfl_manipulation_toolbox/meshes/camera/hand_camera_mount.dae" scale="0.001 0.001 0.001"/></geometry></visual><collision><origin xyz="0 -0.0417 0.0105"/><geometry><box size="0.170 0.225 0.110"/></geometry></collision></link><joint name="camera_mount_joint" type="fixed"><origin xyz="0.05 0 0.10" rpy="0 0 0"/><parent link="link_6"/><child link="camera_mount"/></joint>
-    <link name="camera_color_optical_frame"/><joint name="camera_optical_joint" type="fixed"><origin rpy="-1.5708 0 -1.5708"/><parent link="camera_mount"/><child link="camera_color_optical_frame"/></joint>
+  <xacro:if value="${tool_id == '2fg14'}">
+    <xacro:if value="${robot_id.startswith('picker')}"><xacro:picker_hand_camera/></xacro:if>
+    <link name="2fg14_body">
+      <inertial><mass value="1.5"/><origin xyz="0 0 0.061"/><inertia ixx="0.003616" ixy="0" ixz="0" iyy="0.004677" iyz="0" izz="0.002269"/></inertial>
+      <!-- Dimension-derived visual model.  Published overall dimensions are
+           155.2 x 115 x 70 mm; the jaw opening shown here is nominal only. -->
+      <visual><origin xyz="0 0 -0.0068"/><geometry><cylinder radius="0.0315" length="0.0136"/></geometry><material name="tool_metal"><color rgba="0.55 0.58 0.62 1"/></material></visual>
+      <visual><origin xyz="0 0 0.0516"/><geometry><box size="0.115 0.070 0.1032"/></geometry><material name="tool_blue"><color rgba="0.04 0.28 0.68 1"/></material></visual>
+      <visual><origin xyz="0 -0.036 0.0516"/><geometry><box size="0.096 0.004 0.070"/></geometry><material name="tool_black"><color rgba="0.025 0.035 0.050 1"/></material></visual>
+      <visual><origin xyz="0 0 0.1092"/><geometry><box size="0.100 0.064 0.012"/></geometry><material name="tool_metal"><color rgba="0.55 0.58 0.62 1"/></material></visual>
+      <visual><origin xyz="-0.044 0 0.1292"/><geometry><box size="0.018 0.050 0.052"/></geometry><material name="tool_metal"><color rgba="0.62 0.65 0.68 1"/></material></visual>
+      <visual><origin xyz="0.044 0 0.1292"/><geometry><box size="0.018 0.050 0.052"/></geometry><material name="tool_metal"><color rgba="0.62 0.65 0.68 1"/></material></visual>
+      <visual><origin xyz="-0.044 0 0.1502"/><geometry><box size="0.024 0.058 0.010"/></geometry><material name="tool_black"><color rgba="0.025 0.035 0.050 1"/></material></visual>
+      <visual><origin xyz="0.044 0 0.1502"/><geometry><box size="0.024 0.058 0.010"/></geometry><material name="tool_black"><color rgba="0.025 0.035 0.050 1"/></material></visual>
+      <collision><origin xyz="0 0 0.0776"/><geometry><box size="0.115 0.070 0.1552"/></geometry></collision>
+    </link>
+    <xacro:if value="${robot_id.startswith('picker')}"><joint name="2fg14_mount" type="fixed"><origin xyz="0 0 0.0136"/><parent link="camera_mount"/><child link="2fg14_body"/></joint></xacro:if>
+    <xacro:unless value="${robot_id.startswith('picker')}"><joint name="2fg14_mount" type="fixed"><origin xyz="0 0 0.0136"/><parent link="link_6"/><child link="2fg14_body"/></joint></xacro:unless>
+    <link name="tool_tcp"/><joint name="2fg14_tcp" type="fixed"><origin xyz="0 0 0.136"/><parent link="2fg14_body"/><child link="tool_tcp"/></joint>
   </xacro:if>
   <xacro:if value="${backend == 'gazebo'}">
